File: pcb/pyramid_clock/pyramid_clock.kicad_pcb (KiCad board)
At the start: 2 copper layers, 151 x 111 mm, 25 parts, among them U1 SEEEDUINO-XIAO-ESP32C3

Commit message: updated design, saved gerber and bom
Routing:
- net Net-(D1-VSS): track 36.9 -> 30.7 mm
